Commit message: Updated

File: evarobotmodel_description/urdf/evarobotmodel.urdf (robot description, URDF)
Before this commit: robot evarobotmodel, 34 links, 33 joints
Links:
- link left_wheeltire_link: geometry collision cylinder length=0.001 radius=0.001; visual mesh filename=package://evarobotmodel_description/meshes/tire.dae scale=1 1 1
- link right_wheeltire_link: geometry collision cylinder length=0.001 radius=0.001; visual mesh filename=package://evarobotmodel_description/meshes/tire.dae
Joints:
- joint left_wheel_joint: origin xyz=0 0.16 -0.119 rpy=0 0 0 -> xyz=0.0 -0.16 -0.119 rpy=0.0 0.0 0.0
- joint right_wheel_joint: origin xyz=0.0 -0.16 -0.119 rpy=0.0 0.0 0.0 -> xyz=0 0.16 -0.119 rpy=0 0 0
